File: maint_board/maint_board.sch (KiCad schematic (older format))
At the start: 2 parts, among them J1 USB_mini_micro_B, J2 4P4C

Commit message: added libs and worked on layout
Parts:
- J1: symbol keyboard_parts:USB_mini_micro_B -> maint_board-rescue:USB_mini_micro_B-keyboard_parts
Connections:
- wire segments 35 -> 33
Changed lines of the file:
@@
 F4 "Row3" O L 6050 2950 50
 F5 "Row4" O L 6050 3050 50
-F6 "Row5" O L 6050 3150 50
 F7 "Col1" O L 6050 3550 50
 F8 "Col2" O L 6050 3650 50
@@
 F11 "Col5" O L 6050 3950 50
 F12 "Col6" O L 6050 4050 50
-F13 "Col7" O L 6050 4150 50
 $EndSheet
 $Comp
@@
 F4 "Row3" I R 5700 2950 50
 F5 "Row4" I R 5700 3050 50
-F6 "Row5" I R 5700 3150 50
 F7 "Col1" I R 5700 3550 50
 F8 "Col2" I R 5700 3650 50
@@
 F11 "Col5" I R 5700 3950 50
 F12 "Col6" I R 5700 4050 50
-F13 "Col7" I R 5700 4150 50
 F14 "usb_D-" I L 4400 3050 50
 F15 "usb_D+" I L 4400 3150 50
@@
 	5700 3050 6050 3050
 Wire Wire Line
-	6050 3150 5700 3150
-Wire Wire Line
 	5700 3550 6050 3550
 Wire Wire Line
@@
 Wire Wire Line
 	6050 4050 5700 4050
-Wire Wire Line
-	5700 4150 6050 4150
 $Sheet
 S 6050 4700 1300 750
@@
 	5700 5000 6050 5000
 $Comp
-L keyboard_parts:USB_mini_micro_B J1
+L maint_board-rescue:USB_mini_micro_B-keyboard_parts J1
 U 1 1 601E1AA5
 P 3150 3100

Commit message: Finiched!
Parts:
- J1: footprint keyboard_parts:USB_miniB_hirose_5S8 -> my_connectors:usb_minib_wm5462ct-nd
Other:
- moved on the sheet: J1
Changed lines of the file:
@@
 F4 "Row3" O L 6050 2950 50
 F5 "Row4" O L 6050 3050 50
-F7 "Col1" O L 6050 3550 50
-F8 "Col2" O L 6050 3650 50
-F9 "Col3" O L 6050 3750 50
-F10 "Col4" O L 6050 3850 50
-F11 "Col5" O L 6050 3950 50
-F12 "Col6" O L 6050 4050 50
+F6 "Col1" O L 6050 3550 50
+F7 "Col2" O L 6050 3650 50
+F8 "Col3" O L 6050 3750 50
+F9 "Col4" O L 6050 3850 50
+F10 "Col5" O L 6050 3950 50
+F11 "Col6" O L 6050 4050 50
 $EndSheet
 $Comp
 L power:GND #PWR013
 U 1 1 6050A70E
-P 3950 3550
-F 0 "#PWR013" H 3950 3300 50  0001 C CNN
-F 1 "GND" V 3955 3422 50  0000 R CNN
-F 2 "" H 3950 3550 50  0001 C CNN
-F 3 "" H 3950 3550 50  0001 C CNN
-	1    3950 3550
+P 3000 2250
+F 0 "#PWR013" H 3000 2000 50  0001 C CNN
+F 1 "GND" V 3005 2122 50  0000 R CNN
+F 2 "" H 3000 2250 50  0001 C CNN
+F 3 "" H 3000 2250 50  0001 C CNN
+	1    3000 2250
 	1    0    0    -1
 $EndComp
@@
 F4 "Row3" I R 5700 2950 50
 F5 "Row4" I R 5700 3050 50
-F7 "Col1" I R 5700 3550 50
-F8 "Col2" I R 5700 3650 50
-F9 "Col3" I R 5700 3750 50
-F10 "Col4" I R 5700 3850 50
-F11 "Col5" I R 5700 3950 50
-F12 "Col6" I R 5700 4050 50
-F14 "usb_D-" I L 4400 3050 50
-F15 "usb_D+" I L 4400 3150 50
-F16 "Vcc" I L 4400 2650 50
-F17 "GND" I L 4400 5250 50
-F18 "DoutLed" O R 5700 5000 50
-F19 "SCL" I L 4400 4700 50
-F20 "SDA" I L 4400 4800 50
+F6 "Col1" I R 5700 3550 50
+F7 "Col2" I R 5700 3650 50
+F8 "Col3" I R 5700 3750 50
+F9 "Col4" I R 5700 3850 50
+F10 "Col5" I R 5700 3950 50
+F11 "Col6" I R 5700 4050 50
+F12 "usb_D-" I L 4400 3150 50
+F13 "usb_D+" I L 4400 3050 50
+F14 "Vcc" I L 4400 2650 50
+F15 "GND" I L 4400 5250 50
+F16 "DoutLed" O R 5700 5000 50
+F17 "SCL" I L 4400 4700 50
+F18 "SDA" I L 4400 4800 50
 $EndSheet
 $Comp
 L power:VCC #PWR03
 U 1 1 601B611E
-P 3950 2850
-F 0 "#PWR03" H 3950 2700 50  0001 C CNN
-F 1 "VCC" V 3967 2978 50  0000 L CNN
-F 2 "" H 3950 2850 50  0001 C CNN
-F 3 "" H 3950 2850 50  0001 C CNN
-	1    3950 2850
-	1    0    0    -1
-$EndComp
-Wire Wire Line
-	3300 2950 3950 2950
-Wire Wire Line
-	3950 2950 3950 2850
-Wire Wire Line
-	3300 3350 3950 3350
-Wire Wire Line
-	3950 3350 3950 3450
-Wire Wire Line
-	3300 3450 3950 3450
-Connection ~ 3950 3450
-Wire Wire Line
-	3950 3450 3950 3550
-NoConn ~ 3300 3250
+P 3950 3350
+F 0 "#PWR03" H 3950 3200 50  0001 C CNN
+F 1 "VCC" V 3967 3478 50  0000 L CNN
+F 2 "" H 3950 3350 50  0001 C CNN
+F 3 "" H 3950 3350 50  0001 C CNN
+	1    3950 3350
+	-1   0    0    1
+$EndComp
+Wire Wire Line
+	3300 3250 3950 3250
+Wire Wire Line
+	3950 3350 3950 3250
+Wire Wire Line
+	3300 2750 3450 2750
+NoConn ~ 3300 2950
 Wire Wire Line
 	6050 2750 5700 2750
@@
 F 0 "J1" H 3037 3391 60  0000 C CNN
 F 1 "USB_mini_micro_B" H 3000 3350 60  0001 C CNN
-F 2 "keyboard_parts:USB_miniB_hirose_5S8" H 3100 3100 60  0001 C CNN
+F 2 "my_connectors:usb_minib_wm5462ct-nd" H 3100 3100 60  0001 C CNN
 F 3 "" H 3100 3100 60  0000 C CNN
 	1    3150 3100
-	1    0    0    -1
-$EndComp
+	1    0    0    1
+$EndComp
+Wire Wire Line
+	3450 2750 3450 2150
+Wire Wire Line
+	3450 2150 3000 2150
+Wire Wire Line
+	3000 2150 3000 2250
+Wire Wire Line
+	3300 2850 3450 2850
+Wire Wire Line
+	3450 2850 3450 2750
+Connection ~ 3450 2750
 $EndSCHEMATC

Commit message: updated submodule
Parts:
- J1: symbol maint_board-rescue:USB_mini_micro_B-keyboard_parts -> maint_board-rescue:USB_mini_micro_B-keyboard_parts-maint_board-rescue
Changed lines of the file:
@@
 	5700 5000 6050 5000
 $Comp
-L maint_board-rescue:USB_mini_micro_B-keyboard_parts J1
+L maint_board-rescue:USB_mini_micro_B-keyboard_parts-maint_board-rescue J1
 U 1 1 601E1AA5
 P 3150 3100

Commit message: removed two leds and fixed recet and usb port
Parts:
- J1: footprint my_connectors:usb_minib_wm5462ct-nd -> TB_connectors:usb_minib_wm5462ct-nd
Changed lines of the file:
@@
 F 0 "J1" H 3037 3391 60  0000 C CNN
 F 1 "USB_mini_micro_B" H 3000 3350 60  0001 C CNN
-F 2 "my_connectors:usb_minib_wm5462ct-nd" H 3100 3100 60  0001 C CNN
+F 2 "TB_connectors:usb_minib_wm5462ct-nd" H 3100 3100 60  0001 C CNN
 F 3 "" H 3100 3100 60  0000 C CNN
 	1    3150 3100

Commit message: this is before I switch to usb C
Parts:
- added D14: 1N4148W, Diode_SMD:D_SOD-323, symbol Diode:1N4148W
- added H1, H2, H3: MountingHole, MountingHole:MountingHole_2.2mm_M2_ISO7380, symbol Mechanical:MountingHole
- added J5: USB_C_Receptacle_USB2.0, Connector_USB:USB_C_Receptacle_Palconn_UTC16-G, symbol Connector:USB_C_Receptacle_USB2.0
- added TP1, TP2: TestPoint_Flag, TestPoint:TestPoint_Pad_1.5x1.5mm, symbol Connector:TestPoint_Flag
- J2: footprint my_connectors:glx-n-44_reverseble -> TB_connectors:glx-n-44_reverseble
Connections:
- net GND: now also TP1.1
- net VCC: now also D14.1 (K), TP2.1; no longer J1.1 (VUSB)
- new net: J5.A1 (GND), J5.A12 (GND), J5.B1 (GND), J5.B12 (GND)
- new net: J5.A4 (VBUS), J5.A9 (VBUS), J5.B4 (VBUS), J5.B9 (VBUS)
- new net mcu/Vbus: D14.2 (A), J1.1 (VUSB)
